File: Hardware/PowerSection.kicad_sch (KiCad schematic)
At the start: 14 parts, among them Q6 MMBT3904, SW5 SS12D11, U1 MT3608

Commit message: Updated KiCAD project.
- Added grouping in schematics.
- Removed unnecessary net names in "LogicSection.kicad_sch".
- Added 330R between +5V and nREG_ENABLE.
- Changed path for 3D models.
Other:
- note removed: "V_{REF} = 0.6V V_{REF_min} = 0.588V V_{REF_max} = 0.612V V_{OUT} = V_{REF} * (1 + R22 / R23) V_{OUT} = 9V → R22 = 14kΩ V_{OUT_min} = 8.82V V_{OUT_max} = 9.18V"
Changed lines of the file:
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@@
 	(title_block
 		(title "Simon")
-		(date "2026-03-20")
+		(date "2026-03-31")
 		(rev "01")
 		(company "Kaffeklubben Labs")
 	)
 	(rectangle
-		(start 14.224 155.448)
-		(end 70.612 195.58)
+		(start 13.97 156.21)
+		(end 71.12 195.58)
 		(stroke
 			(width 0)
@@
 		)
 	)
-	(text "V_{REF} = 0.6V\nV_{REF_min} = 0.588V\nV_{REF_max} = 0.612V\n\n\nV_{OUT} = V_{REF} * (1 + R22 / R23)\n\nV_{OUT} = 9V → R22 = 14kΩ\n\nV_{OUT_min} = 8.82V\nV_{OUT_max} = 9.18V"
-		(exclude_from_sim no)
-		(at 17.272 159.004 0)
-		(effects
-			(font
-				(size 1.27 1.27)
-			)
-			(justify left top)
-		)
-	)
 	(text_box "Step-Up Converter Sizing"
 		(exclude_from_sim no)
-		(at 14.224 152.654 0)
-		(size 56.388 2.794)
+		(at 13.97 152.4 0)
+		(size 57.15 3.81)
 		(margins 0.9525 0.9525 0.9525 0.9525)
 		(stroke
@@
 		(effects
 			(font
-				(face "Century Gothic")
+				(face "Consolas")
 				(size 1.27 1.27)
 				(bold yes)
@@
 		)
 	)
+	(text_box "V_{REF} = 0.6V\nV_{REF_min} = 0.588V\nV_{REF_max} = 0.612V\n\n\nV_{OUT} = V_{REF} * (1 + R22 / R23)\n\nV_{OUT} = 9V → R22 = 14kΩ\n\nV_{OUT_min} = 8.82V\nV_{OUT_max} = 9.18V"
+		(exclude_from_sim no)
+		(at 15.24 157.48 0)
+		(size 54.61 36.83)
+		(margins 0.9525 0.9525 0.9525 0.9525)
+		(stroke
+			(width -0.0001)
+			(type solid)
+		)
+		(fill
+			(type none)
+		)
+		(effects
+			(font
+				(face "Consolas")
+				(size 1.27 1.27)
+			)
+			(justify left top)
+		)
+	)
