File: Hardware/Simon.kicad_pcb (KiCad board)
At the start: 2 copper layers, 100 x 100 mm, 69 parts, among them J1 Conn_01x03, J2 Conn_01x03, J3 Conn_01x02, Q1 MMBT3904, Q2 MMBT3904, Q3 MMBT3904, Q4 MMBT3904, Q5 MMBT3904, Q6 MMBT3904, SW1 SW_Push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

Commit message: Updated KiCAD project.
- Added grouping in schematics.
- Removed unnecessary net names in "LogicSection.kicad_sch".
- Added 330R between +5V and nREG_ENABLE.
- Changed path for 3D models.
Parts:
- added R28: 330, Resistor_SMD:R_0805_2012Metric, F.Cu at (122.2, 62.7)
- H1, H2, H3, H4, H5, H6, H7: value MountingHole -> M3 (3.2mm)
- moved R25 4.37 mm to (124.0, 58.5), turned to 90 degrees
- moved R26 0.16 mm to (122.2, 64.7)
Connections:
- net /Logic Section/POT renamed /Input Section/POTENTIOMETER
- net /Logic Section/SWITCH_0 renamed /Input Section/SWITCH_0
- net /Logic Section/SWITCH_1 renamed /Input Section/SWITCH_1
- net /Logic Section/SWITCH_2 renamed /Input Section/SWITCH_2
- net /Logic Section/SWITCH_3 renamed /Input Section/SWITCH_3
- R26 pad 1: +5V -> /Logic Section/~{REG_ENABLE}
- SW5 pad MP: GND -> (no net)
Routing:
- net Net-(D5-A): track 10.9 -> 0.00 mm
- net Net-(U1-FB): track 4.97 -> 0.07 mm
- net /Logic Section/~{REG_ENABLE}: track 0.00 -> 2.76 mm
- net +5V: track 248.4 -> 246.7 mm
- net Net-(D6-K): track 3.32 -> 2.77 mm
- net GND: track 4.47 -> 4.11 mm, vias 3 -> 7
- added copper zone on F.Cu, net Net-(D5-A)
- added copper zone on F.Cu, net Net-(U1-FB)
Other:
- board text added: "LEVEL"
- board text removed: "DIFFICULTY"
